Commit message: complete urdf model of p3dx

File: src/pioneer-p3dx/p3dx_urdf_model/defs/pioneer3dx.urdf (robot description, URDF)
Before this commit: robot pioneer3dx, 11 links, 10 joints
Links:
- removed link back_sonar
- removed link base_link
- removed link center_hubcap
- removed link center_wheel
- removed link front_sonar
- removed link p3dx_left_hubcap
- removed link p3dx_left_wheel
- removed link p3dx_right_hubcap
- removed link p3dx_right_wheel
- removed link swivel
- removed link top_plate
- added link XX/accelerometerSensors/sensor0, mass 0.0001; visual box size=0.1 0.1 0.1
- added link XX/base/joint0; visual mesh filename=package://p3dx_urdf_model/meshes/p3dx_meshes/left_wheel.stl
- added link XX/base/joint1; visual mesh filename=package://p3dx_urdf_model/meshes/p3dx_meshes/right_wheel.stl
- added link XX/base_link, mass 31.1; collision mesh filename=package://p3dx_urdf_model/meshes/p3dx_meshes/chassis.stl; visual mesh filename=package://p3dx_urdf_model/meshes/p3dx_meshes/chassis.stl
- added link XX/bumperSensors/sensor0, mass 0.0001
- added link XX/bumperSensors/sensor1, mass 0.0001
- added link XX/bumperSensors/sensor2, mass 0.0001
- added link XX/bumperSensors/sensor3, mass 0.0001
- added link XX/bumperSensors/sensor4, mass 0.0001
- added link XX/bumperSensors/sensor5, mass 0.0001
- added link XX/bumperSensors/sensor6, mass 0.0001
- added link XX/bumperSensors/sensor7, mass 0.0001
- added link XX/bumperSensors/sensor8, mass 0.0001
- added link XX/bumperSensors/sensor9, mass 0.0001
- added link XX/cameraSensors/sensor0, mass 0.0001; visual box size=0.1 0.1 0.1
- added link XX/center_hubcap, mass 0.01; collision box size=0.05 0.05 0.05; visual mesh filename=package://p3dx_urdf_model/meshes/p3dx_meshes/center_hubcap.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
- added link XX/center_wheel, mass 0.1; collision cylinder length=0.01 radius=0.0375; visual mesh filename=package://p3dx_urdf_model/meshes/p3dx_meshes/center_wheel.s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
- added link XX/gyroSensors/sensor0, mass 0.0001; visual box size=0.1 0.1 0.1
- added link XX/laserSensors/sensor0, mass 0.0001; visual box size=0.1 0.1 0.1
- added link XX/left_hub; collision cylinder length=0.01 radius=0.09; visual mesh filename=package://p3dx_urdf_model/meshes/p3dx_meshes/left_hubcap.stl
- added link XX/right_hub; collision cylinder length=0.01 radius=0.09; visual mesh filename=package://p3dx_urdf_model/meshes/p3dx_meshes/right_hubcap.s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
- added link XX/swivel, mass 0.1; collision box size=0 0 0; visual mesh filename=package://p3dx_urdf_model/meshes/p3dx_meshes/swivel.stl
- added link XX/top_plate, mass 0.01; visual mesh filename=package://p3dx_urdf_model/meshes/p3dx_meshes/top.stl
- added link XX/ultrasonicSensors/sensor0, mass 0.0001
- added link XX/ultrasonicSensors/sensor1, mass 0.0001
- added link XX/ultrasonicSensors/sensor10, mass 0.0001
- added link XX/ultrasonicSensors/sensor11, mass 0.0001
- added link XX/ultrasonicSensors/sensor12, mass 0.0001
- added link XX/ultrasonicSensors/sensor13, mass 0.0001
- added link XX/ultrasonicSensors/sensor14, mass 0.0001
- added link XX/ultrasonicSensors/sensor15, mass 0.0001
- added link XX/ultrasonicSensors/sensor2, mass 0.0001
- added link XX/ultrasonicSensors/sensor3, mass 0.0001
- added link XX/ultrasonicSensors/sensor4, mass 0.0001
- added link XX/ultrasonicSensors/sensor5, mass 0.0001
- added link XX/ultrasonicSensors/sensor6, mass 0.0001
- added link XX/ultrasonicSensors/sensor7, mass 0.0001
- added link XX/ultrasonicSensors/sensor8, mass 0.0001
- added link XX/ultrasonicSensors/sensor9, mass 0.0001
Joints:
- removed joint base_back_joint
- removed joint base_front_joint
- removed joint base_left_hubcap_joint
- removed joint base_left_wheel_joint
- removed joint base_right_hubcap_joint
- removed joint base_right_wheel_joint
- removed joint base_swivel_joint
- removed joint base_top_joint
- removed joint center_wheel_joint
- removed joint swivel_hubcap_joint
- added joint XX/accelerometerSensors/0_joint: type fixed, parent XX/top_plate, child XX/accelerometerSensors/sensor0, origin xyz=0 0 0.0 rpy=0 0 0
- added joint XX/base/joint0: type fixed, parent XX/left_hub, child XX/base/joint0, origin xyz=0 0 0 rpy=0 0 0
- added joint XX/base/joint1: type fixed, parent XX/right_hub, child XX/base/joint1, origin xyz=0 0 0 rpy=0 0 0
- added joint XX/base_swivel_joint: type fixed, parent XX/base_link, child XX/swivel, origin xyz=-0.185 0 0.055 rpy=0 0 0, limit effort=100 velocity=100
- added joint XX/base_top_joint: type fixed, parent XX/base_link, child XX/top_plate, origin xyz=-0.0 0 0.24 rpy=0 0 0
- added joint XX/bumperSensors/0_joint: type fixed, parent XX/base_link, child XX/bumperSensors/sensor0, origin xyz=0.1767 -0.17 0.0681 rpy=0 0 -0.9498
- added joint XX/bumperSensors/1_joint: type fixed, parent XX/base_link, child XX/bumperSensors/sensor1, origin xyz=0.2377 -0.0909 0.0681 rpy=0 0 -0.339
- added joint XX/bumperSensors/2_joint: type fixed, parent XX/base_link, child XX/bumperSensors/sensor2, origin xyz=0.2549 0 0.0681 rpy=0 0 0
- added joint XX/bumperSensors/3_joint: type fixed, parent XX/base_link, child XX/bumperSensors/sensor3, origin xyz=0.2377 0.0909 0.0681 rpy=0 0 0.3535
- added joint XX/bumperSensors/4_joint: type fixed, parent XX/base_link, child XX/bumperSensors/sensor4, origin xyz=0.1767 0.17 0.0681 rpy=0 0 0.9701
- added joint XX/bumperSensors/5_joint: type fixed, parent XX/base_link, child XX/bumperSensors/sensor5, origin xyz=-0.1476 0.1712 0.0681 rpy=0 0 2.0173
- added joint XX/bumperSensors/6_joint: type fixed, parent XX/base_link, child XX/bumperSensors/sensor6, origin xyz=-0.2259 0.0978 0.0681 rpy=0 0 2.6281
- added joint XX/bumperSensors/7_joint: type fixed, parent XX/base_link, child XX/bumperSensors/sensor7, origin xyz=-0.2553 0 0.0681 rpy=0 0 -3.1416
- added joint XX/bumperSensors/8_joint: type fixed, parent XX/base_link, child XX/bumperSensors/sensor8, origin xyz=-0.2259 -0.0978 0.0681 rpy=0 0 -2.6079
- added joint XX/bumperSensors/9_joint: type fixed, parent XX/base_link, child XX/bumperSensors/sensor9, origin xyz=-0.1476 -0.1712 0.0681 rpy=0 0 -1.997
- added joint XX/cameraSensors/0_joint: type fixed, parent XX/top_plate, child XX/cameraSensors/sensor0, origin xyz=0.1498 0 0.001 rpy=1.5708 0 1.5708
- added joint XX/center_wheel_joint: type fixed, parent XX/center_wheel, child XX/center_hubcap, origin xyz=-0.0035 0 -0.001 rpy=0 0 0
- added joint XX/gyroSensors/0_joint: type fixed, parent XX/top_plate, child XX/gyroSensors/sensor0, origin xyz=0 0 0.0 rpy=0 0 0
- added joint XX/laserSensors/0_joint: type fixed, parent XX/top_plate, child XX/laserSensors/sensor0, origin xyz=0.1498 0 0.05 rpy=0 0 0
- added joint XX/left_hub_joint: type fixed, parent XX/base_link, child XX/left_hub, origin xyz=0 0.15 0.08 rpy=0 0 0, axis 0 1 0
- added joint XX/right_hub_joint: type fixed, parent XX/base_link, child XX/right_hub, origin xyz=0 -0.15 0.08 rpy=0 0 0, axis 0 1 0
- added joint XX/swivel_hubcap_joint: type fixed, parent XX/swivel, child XX/center_wheel, origin xyz=-0.026 0 -0.016 rpy=0 0 0, axis 0 1 0, limit effort=100 velocity=100
- added joint XX/ultrasonicSensors/0_joint: type fixed, parent XX/base_link, child XX/ultrasonicSensors/sensor0, origin xyz=0.1064 -0.1381 0.21 rpy=0 0 -1.5708
- added joint XX/ultrasonicSensors/10_joint: type fixed, parent XX/base_link, child XX/ultrasonicSensors/sensor10, origin xyz=-0.1946 0.0785 0.21 rpy=0 0 2.618
- added joint XX/ultrasonicSensors/11_joint: type fixed, parent XX/base_link, child XX/ultrasonicSensors/sensor11, origin xyz=-0.2132 0.0273 0.21 rpy=0 0 2.9663
- added joint XX/ultrasonicSensors/12_joint: type fixed, parent XX/base_link, child XX/ultrasonicSensors/sensor12, origin xyz=-0.2132 -0.0273 0.21 rpy=0 0 2.9663
- added joint XX/ultrasonicSensors/13_joint: type fixed, parent XX/base_link, child XX/ultrasonicSensors/sensor13, origin xyz=-0.1946 -0.0785 0.21 rpy=0 0 -2.618
- added joint XX/ultrasonicSensors/14_joint: type fixed, parent XX/base_link, child XX/ultrasonicSensors/sensor14, origin xyz=-0.1595 -0.1202 0.21 rpy=0 0 -2.2693
- added joint XX/ultrasonicSensors/15_joint: type fixed, parent XX/base_link, child XX/ultrasonicSensors/sensor15, origin xyz=-0.1103 -0.1382 0.21 rpy=0 0 -1.5708
- added joint XX/ultrasonicSensors/1_joint: type fixed, parent XX/base_link, child XX/ultrasonicSensors/sensor1, origin xyz=0.1555 -0.1202 0.21 rpy=0 0 -0.8727
- added joint XX/ultrasonicSensors/2_joint: type fixed, parent XX/base_link, child XX/ultrasonicSensors/sensor2, origin xyz=0.1906 -0.0785 0.21 rpy=0 0 -0.5236
- added joint XX/ultrasonicSensors/3_joint: type fixed, parent XX/base_link, child XX/ultrasonicSensors/sensor3, origin xyz=0.2092 -0.0273 0.21 rpy=0 0 -0.1745
- added joint XX/ultrasonicSensors/4_joint: type fixed, parent XX/base_link, child XX/ultrasonicSensors/sensor4, origin xyz=0.2092 0.0273 0.21 rpy=0 0 0.1745
- added joint XX/ultrasonicSensors/5_joint: type fixed, parent XX/base_link, child XX/ultrasonicSensors/sensor5, origin xyz=0.1906 0.0831 0.21 rpy=0 0 0.5236
- added joint XX/ultrasonicSensors/6_joint: type fixed, parent XX/base_link, child XX/ultrasonicSensors/sensor6, origin xyz=0.1554 0.1251 0.21 rpy=0 0 0.8727
- added joint XX/ultrasonicSensors/7_joint: type fixed, parent XX/base_link, child XX/ultrasonicSensors/sensor7, origin xyz=0.1064 0.1382 0.21 rpy=0 0 1.5708
- added joint XX/ultrasonicSensors/8_joint: type fixed, parent XX/base_link, child XX/ultrasonicSensors/sensor8, origin xyz=-0.1103 0.1382 0.21 rpy=0 0 1.5708
- added joint XX/ultrasonicSensors/9_joint: type fixed, parent XX/base_link, child XX/ultrasonicSensors/sensor9, origin xyz=-0.1595 0.1203 0.21 rpy=0 0 2.2689

File: src/pioneer-p3dx/p3dx_urdf_model/defs/pioneer3dx.xacro (robot description, xacro)
@@ -5,5 +5,5 @@
 	   xmlns:xacro="http://ros.org/wiki/xacro"
 	   name="pioneer3dx">
-	<include filename="$(find p2os_urdf)/defs/pioneer3dx_body.xacro"/>
+	<xacro:include filename="$(find p3dx_urdf_model)/defs/pioneer3dx_body.xacro" />
 	<!-- <xacro:right_wheel_joint suffix="" reflect="1"/>
 	<xacro:left_wheel_joint suffix="" reflect="-1"/>
