Commit message: changes to urdf file

File: src/pioneer-p3dx/p3dx_urdf_model/defs/pioneer3dx.urdf (robot description, URDF)
Before this commit: robot pioneer3dx, 39 links, 38 joints
Links:
- removed link 0/accelerometerSensors/sensor0
- removed link 0/base/joint0
- removed link 0/base/joint1
- removed link 0/base_link
- removed link 0/bumperSensors/sensor0
- removed link 0/bumperSensors/sensor1
- removed link 0/bumperSensors/sensor2
- removed link 0/bumperSensors/sensor3
- removed link 0/bumperSensors/sensor4
- removed link 0/bumperSensors/sensor5
- removed link 0/bumperSensors/sensor6
- removed link 0/bumperSensors/sensor7
- removed link 0/bumperSensors/sensor8
- removed link 0/bumperSensors/sensor9
- removed link 0/cameraSensors/sensor0
- removed link 0/center_hubcap
- removed link 0/center_wheel
- removed link 0/gyroSensors/sensor0
- removed link 0/laserSensors/sensor0
- removed link 0/left_hub
- removed link 0/right_hub
- removed link 0/swivel
- removed link 0/top_plate
- removed link 0/ultrasonicSensors/sensor0
- removed link 0/ultrasonicSensors/sensor1
- removed link 0/ultrasonicSensors/sensor10
- removed link 0/ultrasonicSensors/sensor11
- removed link 0/ultrasonicSensors/sensor12
- removed link 0/ultrasonicSensors/sensor13
- removed link 0/ultrasonicSensors/sensor14
- removed link 0/ultrasonicSensors/sensor15
- removed link 0/ultrasonicSensors/sensor2
- removed link 0/ultrasonicSensors/sensor3
- removed link 0/ultrasonicSensors/sensor4
- removed link 0/ultrasonicSensors/sensor5
- removed link 0/ultrasonicSensors/sensor6
- removed link 0/ultrasonicSensors/sensor7
- removed link 0/ultrasonicSensors/sensor8
- removed link 0/ultrasonicSensors/sensor9
- added link accelerometerSensors/sensor0, mass 0.0001; visual box size=0.1 0.1 0.1
- added link base/joint0; visual mesh filename=package://p3dx_urdf_model/meshes/p3dx_meshes/left_wheel.stl
- added link base/joint1; visual mesh filename=package://p3dx_urdf_model/meshes/p3dx_meshes/right_wheel.stl
- added link base_link, mass 31.1; collision mesh filename=package://p3dx_urdf_model/meshes/p3dx_meshes/chassis.stl; visual mesh filename=package://p3dx_urdf_model/meshes/p3dx_meshes/chassis.stl
- added link bumperSensors/sensor0, mass 0.0001
- added link bumperSensors/sensor1, mass 0.0001
- added link bumperSensors/sensor2, mass 0.0001
- added link bumperSensors/sensor3, mass 0.0001
- added link bumperSensors/sensor4, mass 0.0001
- added link bumperSensors/sensor5, mass 0.0001
- added link bumperSensors/sensor6, mass 0.0001
- added link bumperSensors/sensor7, mass 0.0001
- added link bumperSensors/sensor8, mass 0.0001
- added link bumperSensors/sensor9, mass 0.0001
- added link cameraSensors/sensor0, mass 0.0001; visual box size=0.1 0.1 0.1
- added link center_hubcap, mass 0.01; collision box size=0.05 0.05 0.05; visual mesh filename=package://p3dx_urdf_model/meshes/p3dx_meshes/center_hubcap.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
- added link center_wheel, mass 0.1; collision cylinder length=0.01 radius=0.0375; visual mesh filename=package://p3dx_urdf_model/meshes/p3dx_meshes/center_wheel.s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
- added link gyroSensors/sensor0, mass 0.0001; visual box size=0.1 0.1 0.1
- added link laserSensors/sensor0, mass 0.0001; visual box size=0.1 0.1 0.1
- added link left_hub; collision cylinder length=0.01 radius=0.09; visual mesh filename=package://p3dx_urdf_model/meshes/p3dx_meshes/left_hubcap.stl
- added link right_hub; collision cylinder length=0.01 radius=0.09; visual mesh filename=package://p3dx_urdf_model/meshes/p3dx_meshes/right_hubcap.s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
- added link swivel, mass 0.1; collision box size=0 0 0; visual mesh filename=package://p3dx_urdf_model/meshes/p3dx_meshes/swivel.stl
- added link top_plate, mass 0.01; visual mesh filename=package://p3dx_urdf_model/meshes/p3dx_meshes/top.stl
- added link ultrasonicSensors/sensor0, mass 0.0001
- added link ultrasonicSensors/sensor1, mass 0.0001
- added link ultrasonicSensors/sensor10, mass 0.0001
- added link ultrasonicSensors/sensor11, mass 0.0001
- added link ultrasonicSensors/sensor12, mass 0.0001
- added link ultrasonicSensors/sensor13, mass 0.0001
- added link ultrasonicSensors/sensor14, mass 0.0001
- added link ultrasonicSensors/sensor15, mass 0.0001
- added link ultrasonicSensors/sensor2, mass 0.0001
- added link ultrasonicSensors/sensor3, mass 0.0001
- added link ultrasonicSensors/sensor4, mass 0.0001
- added link ultrasonicSensors/sensor5, mass 0.0001
- added link ultrasonicSensors/sensor6, mass 0.0001
- added link ultrasonicSensors/sensor7, mass 0.0001
- added link ultrasonicSensors/sensor8, mass 0.0001
- added link ultrasonicSensors/sensor9, mass 0.0001
Joints:
- removed joint 0/accelerometerSensors/0_joint
- removed joint 0/base/joint0
- removed joint 0/base/joint1
- removed joint 0/base_swivel_joint
- removed joint 0/base_top_joint
- removed joint 0/bumperSensors/0_joint
- removed joint 0/bumperSensors/1_joint
- removed joint 0/bumperSensors/2_joint
- removed joint 0/bumperSensors/3_joint
- removed joint 0/bumperSensors/4_joint
- removed joint 0/bumperSensors/5_joint
- removed joint 0/bumperSensors/6_joint
- removed joint 0/bumperSensors/7_joint
- removed joint 0/bumperSensors/8_joint
- removed joint 0/bumperSensors/9_joint
- removed joint 0/cameraSensors/0_joint
- removed joint 0/center_wheel_joint
- removed joint 0/gyroSensors/0_joint
- removed joint 0/laserSensors/0_joint
- removed joint 0/left_hub_joint
- removed joint 0/right_hub_joint
- removed joint 0/swivel_hubcap_joint
- removed joint 0/ultrasonicSensors/0_joint
- removed joint 0/ultrasonicSensors/10_joint
- removed joint 0/ultrasonicSensors/11_joint
- removed joint 0/ultrasonicSensors/12_joint
- removed joint 0/ultrasonicSensors/13_joint
- removed joint 0/ultrasonicSensors/14_joint
- removed joint 0/ultrasonicSensors/15_joint
- removed joint 0/ultrasonicSensors/1_joint
- removed joint 0/ultrasonicSensors/2_joint
- removed joint 0/ultrasonicSensors/3_joint
- removed joint 0/ultrasonicSensors/4_joint
- removed joint 0/ultrasonicSensors/5_joint
- removed joint 0/ultrasonicSensors/6_joint
- removed joint 0/ultrasonicSensors/7_joint
- removed joint 0/ultrasonicSensors/8_joint
- removed joint 0/ultrasonicSensors/9_joint
- added joint accelerometerSensors/0_joint: type fixed, parent top_plate, child accelerometerSensors/sensor0, origin xyz=0 0 0.0 rpy=0 0 0
- added joint base/joint0: type fixed, parent left_hub, child base/joint0, origin xyz=0 0 0 rpy=0 0 0
- added joint base/joint1: type fixed, parent right_hub, child base/joint1, origin xyz=0 0 0 rpy=0 0 0
- added joint base_swivel_joint: type fixed, parent base_link, child swivel, origin xyz=-0.185 0 0.055 rpy=0 0 0, limit effort=100 velocity=100
- added joint base_top_joint: type fixed, parent base_link, child top_plate, origin xyz=-0.0 0 0.24 rpy=0 0 0
- added joint bumperSensors/0_joint: type fixed, parent base_link, child bumperSensors/sensor0, origin xyz=0.1767 -0.17 0.0681 rpy=0 0 -0.9498
- added joint bumperSensors/1_joint: type fixed, parent base_link, child bumperSensors/sensor1, origin xyz=0.2377 -0.0909 0.0681 rpy=0 0 -0.339
- added joint bumperSensors/2_joint: type fixed, parent base_link, child bumperSensors/sensor2, origin xyz=0.2549 0 0.0681 rpy=0 0 0
- added joint bumperSensors/3_joint: type fixed, parent base_link, child bumperSensors/sensor3, origin xyz=0.2377 0.0909 0.0681 rpy=0 0 0.3535
- added joint bumperSensors/4_joint: type fixed, parent base_link, child bumperSensors/sensor4, origin xyz=0.1767 0.17 0.0681 rpy=0 0 0.9701
- added joint bumperSensors/5_joint: type fixed, parent base_link, child bumperSensors/sensor5, origin xyz=-0.1476 0.1712 0.0681 rpy=0 0 2.0173
- added joint bumperSensors/6_joint: type fixed, parent base_link, child bumperSensors/sensor6, origin xyz=-0.2259 0.0978 0.0681 rpy=0 0 2.6281
- added joint bumperSensors/7_joint: type fixed, parent base_link, child bumperSensors/sensor7, origin xyz=-0.2553 0 0.0681 rpy=0 0 -3.1416
- added joint bumperSensors/8_joint: type fixed, parent base_link, child bumperSensors/sensor8, origin xyz=-0.2259 -0.0978 0.0681 rpy=0 0 -2.6079
- added joint bumperSensors/9_joint: type fixed, parent base_link, child bumperSensors/sensor9, origin xyz=-0.1476 -0.1712 0.0681 rpy=0 0 -1.997
- added joint cameraSensors/0_joint: type fixed, parent top_plate, child cameraSensors/sensor0, origin xyz=0.1498 0 0.001 rpy=1.5708 0 1.5708
- added joint center_wheel_joint: type fixed, parent center_wheel, child center_hubcap, origin xyz=-0.0035 0 -0.001 rpy=0 0 0
- added joint gyroSensors/0_joint: type fixed, parent top_plate, child gyroSensors/sensor0, origin xyz=0 0 0.0 rpy=0 0 0
- added joint laserSensors/0_joint: type fixed, parent top_plate, child laserSensors/sensor0, origin xyz=0.1498 0 0.05 rpy=0 0 0
- added joint left_hub_joint: type fixed, parent base_link, child left_hub, origin xyz=0 0.15 0.08 rpy=0 0 0, axis 0 1 0
- added joint right_hub_joint: type fixed, parent base_link, child right_hub, origin xyz=0 -0.15 0.08 rpy=0 0 0, axis 0 1 0
- added joint swivel_hubcap_joint: type fixed, parent swivel, child center_wheel, origin xyz=-0.026 0 -0.016 rpy=0 0 0, axis 0 1 0, limit effort=100 velocity=100
- added joint ultrasonicSensors/0_joint: type fixed, parent base_link, child ultrasonicSensors/sensor0, origin xyz=0.1064 -0.1381 0.21 rpy=0 0 -1.5708
- added joint ultrasonicSensors/10_joint: type fixed, parent base_link, child ultrasonicSensors/sensor10, origin xyz=-0.1946 0.0785 0.21 rpy=0 0 2.618
- added joint ultrasonicSensors/11_joint: type fixed, parent base_link, child ultrasonicSensors/sensor11, origin xyz=-0.2132 0.0273 0.21 rpy=0 0 2.9663
- added joint ultrasonicSensors/12_joint: type fixed, parent base_link, child ultrasonicSensors/sensor12, origin xyz=-0.2132 -0.0273 0.21 rpy=0 0 2.9663
- added joint ultrasonicSensors/13_joint: type fixed, parent base_link, child ultrasonicSensors/sensor13, origin xyz=-0.1946 -0.0785 0.21 rpy=0 0 -2.618
- added joint ultrasonicSensors/14_joint: type fixed, parent base_link, child ultrasonicSensors/sensor14, origin xyz=-0.1595 -0.1202 0.21 rpy=0 0 -2.2693
- added joint ultrasonicSensors/15_joint: type fixed, parent base_link, child ultrasonicSensors/sensor15, origin xyz=-0.1103 -0.1382 0.21 rpy=0 0 -1.5708
- added joint ultrasonicSensors/1_joint: type fixed, parent base_link, child ultrasonicSensors/sensor1, origin xyz=0.1555 -0.1202 0.21 rpy=0 0 -0.8727
- added joint ultrasonicSensors/2_joint: type fixed, parent base_link, child ultrasonicSensors/sensor2, origin xyz=0.1906 -0.0785 0.21 rpy=0 0 -0.5236
- added joint ultrasonicSensors/3_joint: type fixed, parent base_link, child ultrasonicSensors/sensor3, origin xyz=0.2092 -0.0273 0.21 rpy=0 0 -0.1745
- added joint ultrasonicSensors/4_joint: type fixed, parent base_link, child ultrasonicSensors/sensor4, origin xyz=0.2092 0.0273 0.21 rpy=0 0 0.1745
- added joint ultrasonicSensors/5_joint: type fixed, parent base_link, child ultrasonicSensors/sensor5, origin xyz=0.1906 0.0831 0.21 rpy=0 0 0.5236
- added joint ultrasonicSensors/6_joint: type fixed, parent base_link, child ultrasonicSensors/sensor6, origin xyz=0.1554 0.1251 0.21 rpy=0 0 0.8727
- added joint ultrasonicSensors/7_joint: type fixed, parent base_link, child ultrasonicSensors/sensor7, origin xyz=0.1064 0.1382 0.21 rpy=0 0 1.5708
- added joint ultrasonicSensors/8_joint: type fixed, parent base_link, child ultrasonicSensors/sensor8, origin xyz=-0.1103 0.1382 0.21 rpy=0 0 1.5708
- added joint ultrasonicSensors/9_joint: type fixed, parent base_link, child ultrasonicSensors/sensor9, origin xyz=-0.1595 0.1203 0.21 rpy=0 0 2.2689

File: src/pioneer-p3dx/p3dx_urdf_model/defs/pioneer3dx.xacro (robot description, xacro)
@@ -6,5 +6,5 @@
 	   name="pioneer3dx">
 	<!--  SET ROBOT NAME -->
-    <property name="robot_id" value="0"/>
+    <property name="robot_id" value=""/>
     <xacro:include filename="$(find p3dx_urdf_model)/defs/pioneer3dx_body.xacro" />
 	<!-- <xacro:right_wheel_joint suffix="" reflect="1"/>

File: src/pioneer-p3dx/p3dx_urdf_model/defs/pioneer3dx_body.xacro (robot description, xacro)
@@ -14,6 +14,5 @@
 		example:
 			0/top_plate
-robot_number is accessed through variable ${robot_id}
--->
+robot_number is accessed through variable ${robot_id}-->
 <robot xmlns:sensor="http://playerstage.sourceforge.net/gazebo/xmlschema/#sensor"
 	   xmlns:controller="http://playerstage.sourceforge.net/gazebo/xmlschema/#controller"
@@ -23,5 +22,5 @@
 	<!-- MACROS -->
 	<xacro:macro name="sonar" params= "id x y z roll pitch yaw" >
-		<link name="${robot_id}/ultrasonicSensors/sensor${id}">
+		<link name="${robot_id}ultrasonicSensors/sensor${id}">
 			<inertial>
 				<mass value="0.0001"/>
@@ -31,16 +30,16 @@
 			</inertial>
 		</link>
-		<gazebo reference="${robot_id}/ultrasonicSensors/sensor${id}">
+		<gazebo reference="${robot_id}ultrasonicSensors/sensor${id}">
 			<material value="Gazebo/Yellow"/>
 		</gazebo>
-		<joint name="${robot_id}/ultrasonicSensors/${id}_joint" type="fixed">
+		<joint name="${robot_id}ultrasonicSensors/${id}_joint" type="fixed">
 			<origin xyz="${x} ${y} ${z}" rpy="${roll} ${pitch} ${yaw}"/>
-			<parent link="${robot_id}/base_link"/>
-			<child link="${robot_id}/ultrasonicSensors/sensor${id}"/>
+			<parent link="${robot_id}base_link"/>
+			<child link="${robot_id}ultrasonicSensors/sensor${id}"/>
 		</joint>
 	</xacro:macro>
 <!--  bumper macro -->
 	<xacro:macro name="bumper" params= "id x y z roll pitch yaw" >
-		<link name="${robot_id}/bumperSensors/sensor${id}">
+		<link name="${robot_id}bumperSensors/sensor${id}">
 			<inertial>
 				<mass value="0.0001"/>
@@ -50,16 +49,16 @@
 			</inertial>
 		</link>
-		<gazebo reference="${robot_id}/bumperSensors/sensor${id}">
+		<gazebo reference="${robot_id}bumperSensors/sensor${id}">
 			<material value="Gazebo/Yellow"/>
 		</gazebo>
-		<joint name="${robot_id}/bumperSensors/${id}_joint" type="fixed">
+		<joint name="${robot_id}bumperSensors/${id}_joint" type="fixed">
 			<origin xyz="${x} ${y} ${z}" rpy="${roll} ${pitch} ${yaw}"/>
-			<parent link="${robot_id}/base_link"/>
-			<child link="${robot_id}/bumperSensors/sensor${id}"/>
+			<parent link="${robot_id}base_link"/>
+			<child link="${robot_id}bumperSensors/sensor${id}"/>
 		</joint>
 	</xacro:macro>
 <!-- *********************************** CHASIS ********************************************** -->
 	<!-- Chassis description -->
-	<link name="${robot_id}/base_link">
+	<link name="${robot_id}base_link">
 		<!-- CHECK THESE VALUES. THEY MAY BE COMPLETELY WRONG. -->
 		<inertial>
@@ -87,9 +86,9 @@
 		</collision>
 	</link>
-	<gazebo reference="${robot_id}/base_link">
+	<gazebo reference="${robot_id}base_link">
 		<material value="Gazebo/Red"/>
 	</gazebo>
 <!-- Top part of the robot -->
-	<link name="${robot_id}/top_plate">
+	<link name="${robot_id}top_plate">
 		<inertial>
 			<mass value="0.01"/>
@@ -108,14 +107,14 @@
 		</visual>
 	</link>
-	<gazebo reference="${robot_id}/top_plate">
+	<gazebo reference="${robot_id}top_plate">
 		<material value="Gazebo/Black"/>
 	</gazebo>
-	<joint name="${robot_id}/base_top_joint" type="fixed">
+	<joint name="${robot_id}base_top_joint" type="fixed">
 		<origin xyz="-0.0 0 0.24" rpy="0 0 0"/>
-		<parent link="${robot_id}/base_link"/>
-		<child link="${robot_id}/top_plate"/>
+		<parent link="${robot_id}base_link"/>
+		<child link="${robot_id}top_plate"/>
 	</joint>
 <!-- ********************************************* CENTER WHEEL****************************************** -->
-<link name="${robot_id}/swivel">
+<link name="${robot_id}swivel">
 		<inertial>
 			<mass value="0.1"/>
@@ -144,5 +143,5 @@
 	</gazebo>
 <!-- Center Wheel + Hubcap -->
-	<link name="${robot_id}/center_hubcap">
+	<link name="${robot_id}center_hubcap">
 		<inertial>
 			<mass value="0.01"/>
@@ -170,5 +169,5 @@
 		<material value="Gazebo/Grey"/>
 	</gazebo>
-	<link name="${robot_id}/center_wheel">
+	<link name="${robot_id}center_wheel">
 		<inertial>
 			<mass value="0.1"/>
@@ -197,13 +196,13 @@
 		<material value="Gazebo/Yellow"/>
 	</gazebo>
-	<joint name="${robot_id}/base_swivel_joint" type="fixed">
+	<joint name="${robot_id}base_swivel_joint" type="fixed">
 		<origin xyz="-0.185 0 0.055" rpy="0 0 0"/>
 		<anchor xyz="0 1 0"/>
     	<limit effort="100" velocity="100" k_velocity="0" />
     	<joint_properties damping="0.0" friction="0.0" />
-		<parent link="${robot_id}/base_link"/>
-		<child link="${robot_id}/swivel"/>
-	</joint>
-	<joint name="${robot_id}/swivel_hubcap_joint" type="fixed">
+		<parent link="${robot_id}base_link"/>
+		<child link="${robot_id}swivel"/>
+	</joint>
+	<joint name="${robot_id}swivel_hubcap_joint" type="fixed">
 		<origin xyz="-0.026 0 -0.016" rpy="0 0 0"/>
 		<axis xyz="0 1 0"/>
@@ -211,14 +210,14 @@
     	<limit effort="100" velocity="100" k_velocity="0" />
     	<joint_properties damping="0.0" friction="0.0" />
-	  	<parent link="${robot_id}/swivel"/>
-		<child link="${robot_id}/center_wheel"/>
-	</joint>
-	<joint name="${robot_id}/center_wheel_joint" type="fixed">
+	  	<parent link="${robot_id}swivel"/>
+		<child link="${robot_id}center_wheel"/>
+	</joint>
+	<joint name="${robot_id}center_wheel_joint" type="fixed">
 		<origin xyz="-0.0035 0 -0.001" rpy="0 0 0"/>
-		<parent link="${robot_id}/center_wheel"/>
-		<child link="${robot_id}/center_hubcap"/>
+		<parent link="${robot_id}center_wheel"/>
+		<child link="${robot_id}center_hubcap"/>
 	</joint>
 	<!-- LEFT WHEEL ***************************************************** -->
-	<link name="${robot_id}/left_hub">
+	<link name="${robot_id}left_hub">
 		<visual>
 			<origin xyz="0 0 0" rpy="0 0 0"/>
@@ -238,5 +237,5 @@
 		</collision>
 	</link>
-	<link name="${robot_id}/base/joint0">
+	<link name="${robot_id}base/joint0">
 		<visual>
 			<origin xyz="0 0 0" rpy="0 0 0"/>
@@ -252,17 +251,17 @@
 		<material value="Gazebo/Black"/>
 	</gazebo>
-	<joint name="${robot_id}/base/joint0" type="fixed">
-		<origin xyz="0 0 0" rpy="0 0 0"/>
-		<parent link="${robot_id}/left_hub"/>
-		<child link="${robot_id}/base/joint0"/>
-	</joint>
-	<joint name="${robot_id}/left_hub_joint" type="fixed">
+	<joint name="${robot_id}base/joint0" type="fixed">
+		<origin xyz="0 0 0" rpy="0 0 0"/>
+		<parent link="${robot_id}left_hub"/>
+		<child link="${robot_id}base/joint0"/>
+	</joint>
+	<joint name="${robot_id}left_hub_joint" type="fixed">
 		<origin xyz="0 0.15 0.08" rpy="0 0 0"/>
-		<parent link="${robot_id}/base_link"/>
-		<child link="${robot_id}/left_hub"/>
+		<parent link="${robot_id}base_link"/>
+		<child link="${robot_id}left_hub"/>
 		<axis xyz="0 1 0"/>
 	</joint>
 <!-- RIGHT WHEEL ***************************************************************** -->
-	<link name="${robot_id}/right_hub">
+	<link name="${robot_id}right_hub">
 		<visual>
 			<origin xyz="0 0 0" rpy="0 0 0"/>
@@ -285,5 +284,5 @@
 		<material value="Gazebo/Yellow"/>
 	</gazebo>
-	<link name="${robot_id}/base/joint1">
+	<link name="${robot_id}base/joint1">
 		<visual>
 			<origin xyz="0 0 0" rpy="0 0 0"/>
@@ -299,13 +298,13 @@
 		<material value="Gazebo/Black"/>
 	</gazebo>
-	<joint name="${robot_id}/base/joint1" type="fixed">
-		<origin xyz="0 0 0" rpy="0 0 0"/>
-		<parent link="${robot_id}/right_hub"/>
-		<child link="${robot_id}/base/joint1"/>
-	</joint>
-	<joint name="${robot_id}/right_hub_joint" type="fixed">
+	<joint name="${robot_id}base/joint1" type="fixed">
+		<origin xyz="0 0 0" rpy="0 0 0"/>
+		<parent link="${robot_id}right_hub"/>
+		<child link="${robot_id}base/joint1"/>
+	</joint>
+	<joint name="${robot_id}right_hub_joint" type="fixed">
 		<origin xyz="0 -0.15 0.08" rpy="0 0 0"/>
-		<parent link="${robot_id}/base_link"/>
-		<child link="${robot_id}/right_hub"/>
+		<parent link="${robot_id}base_link"/>
+		<child link="${robot_id}right_hub"/>
 		<axis xyz="0 1 0"/>
 	</joint>
@@ -346,5 +345,5 @@
 	<bumper id="9" x="-0.1476" y="-0.1712" z="${bumper_height}" roll="0" pitch="0" yaw="${-1.5708-0.4262}" />
 <!-- ************************************************ LASER SCANER ********************************-->
-	<link name="${robot_id}/laserSensors/sensor0">
+	<link name="${robot_id}laserSensors/sensor0">
 		<inertial>
 			<mass value="0.0001"/>
@@ -363,14 +362,14 @@
     	</visual>
 	</link>
-	<gazebo reference="${robot_id}/laserSensors/sensor0">
+	<gazebo reference="${robot_id}laserSensors/sensor0">
 		<material value="Gazebo/Blue"/>
 	</gazebo>
-	<joint name="${robot_id}/laserSensors/0_joint" type="fixed">
+	<joint name="${robot_id}laserSensors/0_joint" type="fixed">
 		<origin xyz="0.1498 0 0.05" rpy="0 0 0"/>
-		<parent link="${robot_id}/top_plate"/>
-		<child link="${robot_id}/laserSensors/sensor0"/>
+		<parent link="${robot_id}top_plate"/>
+		<child link="${robot_id}laserSensors/sensor0"/>
 	</joint>
 	<!-- ************************************************ CAMERA ********************************-->
-	<link name="${robot_id}/cameraSensors/sensor0">
+	<link name="${robot_id}cameraSensors/sensor0">
 		<inertial>
 			<mass value="0.0001"/>
@@ -389,14 +388,14 @@
     	</visual>
 	</link>
-	<gazebo reference="${robot_id}/cameraSensors/sensor0">
+	<gazebo reference="${robot_id}cameraSensors/sensor0">
 		<material value="Gazebo/Blue"/>
 	</gazebo>
-	<joint name="${robot_id}/cameraSensors/0_joint" type="fixed">
+	<joint name="${robot_id}cameraSensors/0_joint" type="fixed">
 		<origin xyz="0.1498 0 0.001" rpy="1.5708 0 1.5708"/>
-		<parent link="${robot_id}/top_plate"/>
-		<child link="${robot_id}/cameraSensors/sensor0"/>
+		<parent link="${robot_id}top_plate"/>
+		<child link="${robot_id}cameraSensors/sensor0"/>
 	</joint>
 	<!-- ************************************************ GYRO ********************************-->
-	<link name="${robot_id}/gyroSensors/sensor0">
+	<link name="${robot_id}gyroSensors/sensor0">
 		<inertial>
 			<mass value="0.0001"/>
@@ -415,14 +414,14 @@
     	</visual>
 	</link>
-	<gazebo reference="${robot_id}/gyroSensors/sensor0">
+	<gazebo reference="${robot_id}gyroSensors/sensor0">
 		<material value="Gazebo/Blue"/>
 	</gazebo>
-	<joint name="${robot_id}/gyroSensors/0_joint" type="fixed">
+	<joint name="${robot_id}gyroSensors/0_joint" type="fixed">
 		<origin xyz="0 0 0.0" rpy="0 0 0"/>
-		<parent link="${robot_id}/top_plate"/>
-		<child link="${robot_id}/gyroSensors/sensor0"/>
+		<parent link="${robot_id}top_plate"/>
+		<child link="${robot_id}gyroSensors/sensor0"/>
 	</joint>
 <!-- ************************************************ ACCELEROMETER ********************************-->
-	<link name="${robot_id}/accelerometerSensors/sensor0">
+	<link name="${robot_id}accelerometerSensors/sensor0">
 		<inertial>
 			<mass value="0.0001"/>
@@ -441,11 +440,11 @@
     	</visual>
 	</link>
-	<gazebo reference="${robot_id}/accelerometerSensors/sensor0">
+	<gazebo reference="${robot_id}accelerometerSensors/sensor0">
 		<material value="Gazebo/Blue"/>
 	</gazebo>
-	<joint name="${robot_id}/accelerometerSensors/0_joint" type="fixed">
+	<joint name="${robot_id}accelerometerSensors/0_joint" type="fixed">
 		<origin xyz="0 0 0.0" rpy="0 0 0"/>
-		<parent link="${robot_id}/top_plate"/>
-		<child link="${robot_id}/accelerometerSensors/sensor0"/>
+		<parent link="${robot_id}top_plate"/>
+		<child link="${robot_id}accelerometerSensors/sensor0"/>
 	</joint>
 	<xacro:macro name="p3dx_gazebo_ext">
