Commit message: Revert "changes to urdf file"
This reverts commit f1edb606f8ce90d60382e3983028824879ccc51d.

	modified:   src/pioneer-p3dx/p3dx_urdf_model/defs/pioneer3dx.xacro
	modified:   src/pioneer-p3dx/p3dx_urdf_model/defs/pioneer3dx_body.xacro
	modified:   src/pioneer-p3dx/p3dx_urdf_model/launch/pioneer3dx_urdf.launch

File: src/pioneer-p3dx/p3dx_urdf_model/defs/pioneer3dx.urdf (robot description, URDF)
Before this commit: robot pioneer3dx, 39 links, 38 joints
Links:
- removed link accelerometerSensors/sensor0
- removed link base/joint0
- removed link base/joint1
- removed link base_link
- removed link bumperSensors/sensor0
- removed link bumperSensors/sensor1
- removed link bumperSensors/sensor2
- removed link bumperSensors/sensor3
- removed link bumperSensors/sensor4
- removed link bumperSensors/sensor5
- removed link bumperSensors/sensor6
- removed link bumperSensors/sensor7
- removed link bumperSensors/sensor8
- removed link bumperSensors/sensor9
- removed link cameraSensors/sensor0
- removed link center_hubcap
- removed link center_wheel
- removed link gyroSensors/sensor0
- removed link laserSensors/sensor0
- removed link left_hub
- removed link right_hub
- removed link swivel
- removed link top_plate
- removed link ultrasonicSensors/sensor0
- removed link ultrasonicSensors/sensor1
- removed link ultrasonicSensors/sensor10
- removed link ultrasonicSensors/sensor11
- removed link ultrasonicSensors/sensor12
- removed link ultrasonicSensors/sensor13
- removed link ultrasonicSensors/sensor14
- removed link ultrasonicSensors/sensor15
- removed link ultrasonicSensors/sensor2
- removed link ultrasonicSensors/sensor3
- removed link ultrasonicSensors/sensor4
- removed link ultrasonicSensors/sensor5
- removed link ultrasonicSensors/sensor6
- removed link ultrasonicSensors/sensor7
- removed link ultrasonicSensors/sensor8
- removed link ultrasonicSensors/sensor9
- added link 0/accelerometerSensors/sensor0, mass 0.0001; visual box size=0.1 0.1 0.1
- added link 0/base/joint0; visual mesh filename=package://p3dx_urdf_model/meshes/p3dx_meshes/left_wheel.stl
- added link 0/base/joint1; visual mesh filename=package://p3dx_urdf_model/meshes/p3dx_meshes/right_wheel.stl
- added link 0/base_link, mass 31.1; collision mesh filename=package://p3dx_urdf_model/meshes/p3dx_meshes/chassis.stl; visual mesh filename=package://p3dx_urdf_model/meshes/p3dx_meshes/chassis.stl
- added link 0/bumperSensors/sensor0, mass 0.0001
- added link 0/bumperSensors/sensor1, mass 0.0001
- added link 0/bumperSensors/sensor2, mass 0.0001
- added link 0/bumperSensors/sensor3, mass 0.0001
- added link 0/bumperSensors/sensor4, mass 0.0001
- added link 0/bumperSensors/sensor5, mass 0.0001
- added link 0/bumperSensors/sensor6, mass 0.0001
- added link 0/bumperSensors/sensor7, mass 0.0001
- added link 0/bumperSensors/sensor8, mass 0.0001
- added link 0/bumperSensors/sensor9, mass 0.0001
- added link 0/cameraSensors/sensor0, mass 0.0001; visual box size=0.1 0.1 0.1
- added link 0/center_hubcap, mass 0.01; collision box size=0.05 0.05 0.05; visual mesh filename=package://p3dx_urdf_model/meshes/p3dx_meshes/center_hubcap.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
- added link 0/center_wheel, mass 0.1; collision cylinder length=0.01 radius=0.0375; visual mesh filename=package://p3dx_urdf_model/meshes/p3dx_meshes/center_wheel.s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
- added link 0/gyroSensors/sensor0, mass 0.0001; visual box size=0.1 0.1 0.1
- added link 0/laserSensors/sensor0, mass 0.0001; visual box size=0.1 0.1 0.1
- added link 0/left_hub; collision cylinder length=0.01 radius=0.09; visual mesh filename=package://p3dx_urdf_model/meshes/p3dx_meshes/left_hubcap.stl
- added link 0/right_hub; collision cylinder length=0.01 radius=0.09; visual mesh filename=package://p3dx_urdf_model/meshes/p3dx_meshes/right_hubcap.s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
- added link 0/swivel, mass 0.1; collision box size=0 0 0; visual mesh filename=package://p3dx_urdf_model/meshes/p3dx_meshes/swivel.stl
- added link 0/top_plate, mass 0.01; visual mesh filename=package://p3dx_urdf_model/meshes/p3dx_meshes/top.stl
- added link 0/ultrasonicSensors/sensor0, mass 0.0001
- added link 0/ultrasonicSensors/sensor1, mass 0.0001
- added link 0/ultrasonicSensors/sensor10, mass 0.0001
- added link 0/ultrasonicSensors/sensor11, mass 0.0001
- added link 0/ultrasonicSensors/sensor12, mass 0.0001
- added link 0/ultrasonicSensors/sensor13, mass 0.0001
- added link 0/ultrasonicSensors/sensor14, mass 0.0001
- added link 0/ultrasonicSensors/sensor15, mass 0.0001
- added link 0/ultrasonicSensors/sensor2, mass 0.0001
- added link 0/ultrasonicSensors/sensor3, mass 0.0001
- added link 0/ultrasonicSensors/sensor4, mass 0.0001
- added link 0/ultrasonicSensors/sensor5, mass 0.0001
- added link 0/ultrasonicSensors/sensor6, mass 0.0001
- added link 0/ultrasonicSensors/sensor7, mass 0.0001
- added link 0/ultrasonicSensors/sensor8, mass 0.0001
- added link 0/ultrasonicSensors/sensor9, mass 0.0001
Joints:
- removed joint accelerometerSensors/0_joint
- removed joint base/joint0
- removed joint base/joint1
- removed joint base_swivel_joint
- removed joint base_top_joint
- removed joint bumperSensors/0_joint
- removed joint bumperSensors/1_joint
- removed joint bumperSensors/2_joint
- removed joint bumperSensors/3_joint
- removed joint bumperSensors/4_joint
- removed joint bumperSensors/5_joint
- removed joint bumperSensors/6_joint
- removed joint bumperSensors/7_joint
- removed joint bumperSensors/8_joint
- removed joint bumperSensors/9_joint
- removed joint cameraSensors/0_joint
- removed joint center_wheel_joint
- removed joint gyroSensors/0_joint
- removed joint laserSensors/0_joint
- removed joint left_hub_joint
- removed joint right_hub_joint
- removed joint swivel_hubcap_joint
- removed joint ultrasonicSensors/0_joint
- removed joint ultrasonicSensors/10_joint
- removed joint ultrasonicSensors/11_joint
- removed joint ultrasonicSensors/12_joint
- removed joint ultrasonicSensors/13_joint
- removed joint ultrasonicSensors/14_joint
- removed joint ultrasonicSensors/15_joint
- removed joint ultrasonicSensors/1_joint
- removed joint ultrasonicSensors/2_joint
- removed joint ultrasonicSensors/3_joint
- removed joint ultrasonicSensors/4_joint
- removed joint ultrasonicSensors/5_joint
- removed joint ultrasonicSensors/6_joint
- removed joint ultrasonicSensors/7_joint
- removed joint ultrasonicSensors/8_joint
- removed joint ultrasonicSensors/9_joint
- added joint 0/accelerometerSensors/0_joint: type fixed, parent 0/top_plate, child 0/accelerometerSensors/sensor0, origin xyz=0 0 0.0 rpy=0 0 0
- added joint 0/base/joint0: type fixed, parent 0/left_hub, child 0/base/joint0, origin xyz=0 0 0 rpy=0 0 0
- added joint 0/base/joint1: type fixed, parent 0/right_hub, child 0/base/joint1, origin xyz=0 0 0 rpy=0 0 0
- added joint 0/base_swivel_joint: type fixed, parent 0/base_link, child 0/swivel, origin xyz=-0.185 0 0.055 rpy=0 0 0, limit effort=100 velocity=100
- added joint 0/base_top_joint: type fixed, parent 0/base_link, child 0/top_plate, origin xyz=-0.0 0 0.24 rpy=0 0 0
- added joint 0/bumperSensors/0_joint: type fixed, parent 0/base_link, child 0/bumperSensors/sensor0, origin xyz=0.1767 -0.17 0.0681 rpy=0 0 -0.9498
- added joint 0/bumperSensors/1_joint: type fixed, parent 0/base_link, child 0/bumperSensors/sensor1, origin xyz=0.2377 -0.0909 0.0681 rpy=0 0 -0.339
- added joint 0/bumperSensors/2_joint: type fixed, parent 0/base_link, child 0/bumperSensors/sensor2, origin xyz=0.2549 0 0.0681 rpy=0 0 0
- added joint 0/bumperSensors/3_joint: type fixed, parent 0/base_link, child 0/bumperSensors/sensor3, origin xyz=0.2377 0.0909 0.0681 rpy=0 0 0.3535
- added joint 0/bumperSensors/4_joint: type fixed, parent 0/base_link, child 0/bumperSensors/sensor4, origin xyz=0.1767 0.17 0.0681 rpy=0 0 0.9701
- added joint 0/bumperSensors/5_joint: type fixed, parent 0/base_link, child 0/bumperSensors/sensor5, origin xyz=-0.1476 0.1712 0.0681 rpy=0 0 2.0173
- added joint 0/bumperSensors/6_joint: type fixed, parent 0/base_link, child 0/bumperSensors/sensor6, origin xyz=-0.2259 0.0978 0.0681 rpy=0 0 2.6281
- added joint 0/bumperSensors/7_joint: type fixed, parent 0/base_link, child 0/bumperSensors/sensor7, origin xyz=-0.2553 0 0.0681 rpy=0 0 -3.1416
- added joint 0/bumperSensors/8_joint: type fixed, parent 0/base_link, child 0/bumperSensors/sensor8, origin xyz=-0.2259 -0.0978 0.0681 rpy=0 0 -2.6079
- added joint 0/bumperSensors/9_joint: type fixed, parent 0/base_link, child 0/bumperSensors/sensor9, origin xyz=-0.1476 -0.1712 0.0681 rpy=0 0 -1.997
- added joint 0/cameraSensors/0_joint: type fixed, parent 0/top_plate, child 0/cameraSensors/sensor0, origin xyz=0.1498 0 0.001 rpy=1.5708 0 1.5708
- added joint 0/center_wheel_joint: type fixed, parent 0/center_wheel, child 0/center_hubcap, origin xyz=-0.0035 0 -0.001 rpy=0 0 0
- added joint 0/gyroSensors/0_joint: type fixed, parent 0/top_plate, child 0/gyroSensors/sensor0, origin xyz=0 0 0.0 rpy=0 0 0
- added joint 0/laserSensors/0_joint: type fixed, parent 0/top_plate, child 0/laserSensors/sensor0, origin xyz=0.1498 0 0.05 rpy=0 0 0
- added joint 0/left_hub_joint: type fixed, parent 0/base_link, child 0/left_hub, origin xyz=0 0.15 0.08 rpy=0 0 0, axis 0 1 0
- added joint 0/right_hub_joint: type fixed, parent 0/base_link, child 0/right_hub, origin xyz=0 -0.15 0.08 rpy=0 0 0, axis 0 1 0
- added joint 0/swivel_hubcap_joint: type fixed, parent 0/swivel, child 0/center_wheel, origin xyz=-0.026 0 -0.016 rpy=0 0 0, axis 0 1 0, limit effort=100 velocity=100
- added joint 0/ultrasonicSensors/0_joint: type fixed, parent 0/base_link, child 0/ultrasonicSensors/sensor0, origin xyz=0.1064 -0.1381 0.21 rpy=0 0 -1.5708
- added joint 0/ultrasonicSensors/10_joint: type fixed, parent 0/base_link, child 0/ultrasonicSensors/sensor10, origin xyz=-0.1946 0.0785 0.21 rpy=0 0 2.618
- added joint 0/ultrasonicSensors/11_joint: type fixed, parent 0/base_link, child 0/ultrasonicSensors/sensor11, origin xyz=-0.2132 0.0273 0.21 rpy=0 0 2.9663
- added joint 0/ultrasonicSensors/12_joint: type fixed, parent 0/base_link, child 0/ultrasonicSensors/sensor12, origin xyz=-0.2132 -0.0273 0.21 rpy=0 0 2.9663
- added joint 0/ultrasonicSensors/13_joint: type fixed, parent 0/base_link, child 0/ultrasonicSensors/sensor13, origin xyz=-0.1946 -0.0785 0.21 rpy=0 0 -2.618
- added joint 0/ultrasonicSensors/14_joint: type fixed, parent 0/base_link, child 0/ultrasonicSensors/sensor14, origin xyz=-0.1595 -0.1202 0.21 rpy=0 0 -2.2693
- added joint 0/ultrasonicSensors/15_joint: type fixed, parent 0/base_link, child 0/ultrasonicSensors/sensor15, origin xyz=-0.1103 -0.1382 0.21 rpy=0 0 -1.5708
- added joint 0/ultrasonicSensors/1_joint: type fixed, parent 0/base_link, child 0/ultrasonicSensors/sensor1, origin xyz=0.1555 -0.1202 0.21 rpy=0 0 -0.8727
- added joint 0/ultrasonicSensors/2_joint: type fixed, parent 0/base_link, child 0/ultrasonicSensors/sensor2, origin xyz=0.1906 -0.0785 0.21 rpy=0 0 -0.5236
- added joint 0/ultrasonicSensors/3_joint: type fixed, parent 0/base_link, child 0/ultrasonicSensors/sensor3, origin xyz=0.2092 -0.0273 0.21 rpy=0 0 -0.1745
- added joint 0/ultrasonicSensors/4_joint: type fixed, parent 0/base_link, child 0/ultrasonicSensors/sensor4, origin xyz=0.2092 0.0273 0.21 rpy=0 0 0.1745
- added joint 0/ultrasonicSensors/5_joint: type fixed, parent 0/base_link, child 0/ultrasonicSensors/sensor5, origin xyz=0.1906 0.0831 0.21 rpy=0 0 0.5236
- added joint 0/ultrasonicSensors/6_joint: type fixed, parent 0/base_link, child 0/ultrasonicSensors/sensor6, origin xyz=0.1554 0.1251 0.21 rpy=0 0 0.8727
- added joint 0/ultrasonicSensors/7_joint: type fixed, parent 0/base_link, child 0/ultrasonicSensors/sensor7, origin xyz=0.1064 0.1382 0.21 rpy=0 0 1.5708
- added joint 0/ultrasonicSensors/8_joint: type fixed, parent 0/base_link, child 0/ultrasonicSensors/sensor8, origin xyz=-0.1103 0.1382 0.21 rpy=0 0 1.5708
- added joint 0/ultrasonicSensors/9_joint: type fixed, parent 0/base_link, child 0/ultrasonicSensors/sensor9, origin xyz=-0.1595 0.1203 0.21 rpy=0 0 2.2689

File: src/pioneer-p3dx/p3dx_urdf_model/defs/pioneer3dx.xacro (robot description, xacro)
@@ -6,5 +6,5 @@
 	   name="pioneer3dx">
 	<!--  SET ROBOT NAME -->
-    <property name="robot_id" value=""/>
+    <property name="robot_id" value="0"/>
     <xacro:include filename="$(find p3dx_urdf_model)/defs/pioneer3dx_body.xacro" />
 	<!-- <xacro:right_wheel_joint suffix="" reflect="1"/>
