Commit message: Revert "changes to urdf file"
This reverts commit f1edb606f8ce90d60382e3983028824879ccc51d.

	modified:   src/pioneer-p3dx/p3dx_urdf_model/defs/pioneer3dx.xacro
	modified:   src/pioneer-p3dx/p3dx_urdf_model/defs/pioneer3dx_body.xacro
	modified:   src/pioneer-p3dx/p3dx_urdf_model/launch/pioneer3dx_urdf.launch

File: src/pioneer-p3dx/p3dx_urdf_model/defs/pioneer3dx_body.xacro (robot description, xacro)
@@ -14,5 +14,6 @@
 		example:
 			0/top_plate
-robot_number is accessed through variable ${robot_id}-->
+robot_number is accessed through variable ${robot_id}
+-->
 <robot xmlns:sensor="http://playerstage.sourceforge.net/gazebo/xmlschema/#sensor"
 	   xmlns:controller="http://playerstage.sourceforge.net/gazebo/xmlschema/#controller"
@@ -22,5 +23,5 @@
 	<!-- MACROS -->
 	<xacro:macro name="sonar" params= "id x y z roll pitch yaw" >
-		<link name="${robot_id}ultrasonicSensors/sensor${id}">
+		<link name="${robot_id}/ultrasonicSensors/sensor${id}">
 			<inertial>
 				<mass value="0.0001"/>
@@ -30,16 +31,16 @@
 			</inertial>
 		</link>
-		<gazebo reference="${robot_id}ultrasonicSensors/sensor${id}">
+		<gazebo reference="${robot_id}/ultrasonicSensors/sensor${id}">
 			<material value="Gazebo/Yellow"/>
 		</gazebo>
-		<joint name="${robot_id}ultrasonicSensors/${id}_joint" type="fixed">
+		<joint name="${robot_id}/ultrasonicSensors/${id}_joint" type="fixed">
 			<origin xyz="${x} ${y} ${z}" rpy="${roll} ${pitch} ${yaw}"/>
-			<parent link="${robot_id}base_link"/>
-			<child link="${robot_id}ultrasonicSensors/sensor${id}"/>
+			<parent link="${robot_id}/base_link"/>
+			<child link="${robot_id}/ultrasonicSensors/sensor${id}"/>
 		</joint>
 	</xacro:macro>
 <!--  bumper macro -->
 	<xacro:macro name="bumper" params= "id x y z roll pitch yaw" >
-		<link name="${robot_id}bumperSensors/sensor${id}">
+		<link name="${robot_id}/bumperSensors/sensor${id}">
 			<inertial>
 				<mass value="0.0001"/>
@@ -49,16 +50,16 @@
 			</inertial>
 		</link>
-		<gazebo reference="${robot_id}bumperSensors/sensor${id}">
+		<gazebo reference="${robot_id}/bumperSensors/sensor${id}">
 			<material value="Gazebo/Yellow"/>
 		</gazebo>
-		<joint name="${robot_id}bumperSensors/${id}_joint" type="fixed">
+		<joint name="${robot_id}/bumperSensors/${id}_joint" type="fixed">
 			<origin xyz="${x} ${y} ${z}" rpy="${roll} ${pitch} ${yaw}"/>
-			<parent link="${robot_id}base_link"/>
-			<child link="${robot_id}bumperSensors/sensor${id}"/>
+			<parent link="${robot_id}/base_link"/>
+			<child link="${robot_id}/bumperSensors/sensor${id}"/>
 		</joint>
 	</xacro:macro>
 <!-- *********************************** CHASIS ********************************************** -->
 	<!-- Chassis description -->
-	<link name="${robot_id}base_link">
+	<link name="${robot_id}/base_link">
 		<!-- CHECK THESE VALUES. THEY MAY BE COMPLETELY WRONG. -->
 		<inertial>
@@ -86,9 +87,9 @@
 		</collision>
 	</link>
-	<gazebo reference="${robot_id}base_link">
+	<gazebo reference="${robot_id}/base_link">
 		<material value="Gazebo/Red"/>
 	</gazebo>
 <!-- Top part of the robot -->
-	<link name="${robot_id}top_plate">
+	<link name="${robot_id}/top_plate">
 		<inertial>
 			<mass value="0.01"/>
@@ -107,14 +108,14 @@
 		</visual>
 	</link>
-	<gazebo reference="${robot_id}top_plate">
+	<gazebo reference="${robot_id}/top_plate">
 		<material value="Gazebo/Black"/>
 	</gazebo>
-	<joint name="${robot_id}base_top_joint" type="fixed">
+	<joint name="${robot_id}/base_top_joint" type="fixed">
 		<origin xyz="-0.0 0 0.24" rpy="0 0 0"/>
-		<parent link="${robot_id}base_link"/>
-		<child link="${robot_id}top_plate"/>
+		<parent link="${robot_id}/base_link"/>
+		<child link="${robot_id}/top_plate"/>
 	</joint>
 <!-- ********************************************* CENTER WHEEL****************************************** -->
-<link name="${robot_id}swivel">
+<link name="${robot_id}/swivel">
 		<inertial>
 			<mass value="0.1"/>
@@ -143,5 +144,5 @@
 	</gazebo>
 <!-- Center Wheel + Hubcap -->
-	<link name="${robot_id}center_hubcap">
+	<link name="${robot_id}/center_hubcap">
 		<inertial>
 			<mass value="0.01"/>
@@ -169,5 +170,5 @@
 		<material value="Gazebo/Grey"/>
 	</gazebo>
-	<link name="${robot_id}center_wheel">
+	<link name="${robot_id}/center_wheel">
 		<inertial>
 			<mass value="0.1"/>
@@ -196,13 +197,13 @@
 		<material value="Gazebo/Yellow"/>
 	</gazebo>
-	<joint name="${robot_id}base_swivel_joint" type="fixed">
+	<joint name="${robot_id}/base_swivel_joint" type="fixed">
 		<origin xyz="-0.185 0 0.055" rpy="0 0 0"/>
 		<anchor xyz="0 1 0"/>
     	<limit effort="100" velocity="100" k_velocity="0" />
     	<joint_properties damping="0.0" friction="0.0" />
-		<parent link="${robot_id}base_link"/>
-		<child link="${robot_id}swivel"/>
-	</joint>
-	<joint name="${robot_id}swivel_hubcap_joint" type="fixed">
+		<parent link="${robot_id}/base_link"/>
+		<child link="${robot_id}/swivel"/>
+	</joint>
+	<joint name="${robot_id}/swivel_hubcap_joint" type="fixed">
 		<origin xyz="-0.026 0 -0.016" rpy="0 0 0"/>
 		<axis xyz="0 1 0"/>
@@ -210,14 +211,14 @@
     	<limit effort="100" velocity="100" k_velocity="0" />
     	<joint_properties damping="0.0" friction="0.0" />
-	  	<parent link="${robot_id}swivel"/>
-		<child link="${robot_id}center_wheel"/>
-	</joint>
-	<joint name="${robot_id}center_wheel_joint" type="fixed">
+	  	<parent link="${robot_id}/swivel"/>
+		<child link="${robot_id}/center_wheel"/>
+	</joint>
+	<joint name="${robot_id}/center_wheel_joint" type="fixed">
 		<origin xyz="-0.0035 0 -0.001" rpy="0 0 0"/>
-		<parent link="${robot_id}center_wheel"/>
-		<child link="${robot_id}center_hubcap"/>
+		<parent link="${robot_id}/center_wheel"/>
+		<child link="${robot_id}/center_hubcap"/>
 	</joint>
 	<!-- LEFT WHEEL ***************************************************** -->
-	<link name="${robot_id}left_hub">
+	<link name="${robot_id}/left_hub">
 		<visual>
 			<origin xyz="0 0 0" rpy="0 0 0"/>
@@ -237,5 +238,5 @@
 		</collision>
 	</link>
-	<link name="${robot_id}base/joint0">
+	<link name="${robot_id}/base/joint0">
 		<visual>
 			<origin xyz="0 0 0" rpy="0 0 0"/>
@@ -251,17 +252,17 @@
 		<material value="Gazebo/Black"/>
 	</gazebo>
-	<joint name="${robot_id}base/joint0" type="fixed">
-		<origin xyz="0 0 0" rpy="0 0 0"/>
-		<parent link="${robot_id}left_hub"/>
-		<child link="${robot_id}base/joint0"/>
-	</joint>
-	<joint name="${robot_id}left_hub_joint" type="fixed">
+	<joint name="${robot_id}/base/joint0" type="fixed">
+		<origin xyz="0 0 0" rpy="0 0 0"/>
+		<parent link="${robot_id}/left_hub"/>
+		<child link="${robot_id}/base/joint0"/>
+	</joint>
+	<joint name="${robot_id}/left_hub_joint" type="fixed">
 		<origin xyz="0 0.15 0.08" rpy="0 0 0"/>
-		<parent link="${robot_id}base_link"/>
-		<child link="${robot_id}left_hub"/>
+		<parent link="${robot_id}/base_link"/>
+		<child link="${robot_id}/left_hub"/>
 		<axis xyz="0 1 0"/>
 	</joint>
 <!-- RIGHT WHEEL ***************************************************************** -->
-	<link name="${robot_id}right_hub">
+	<link name="${robot_id}/right_hub">
 		<visual>
 			<origin xyz="0 0 0" rpy="0 0 0"/>
@@ -284,5 +285,5 @@
 		<material value="Gazebo/Yellow"/>
 	</gazebo>
-	<link name="${robot_id}base/joint1">
+	<link name="${robot_id}/base/joint1">
 		<visual>
 			<origin xyz="0 0 0" rpy="0 0 0"/>
@@ -298,13 +299,13 @@
 		<material value="Gazebo/Black"/>
 	</gazebo>
-	<joint name="${robot_id}base/joint1" type="fixed">
-		<origin xyz="0 0 0" rpy="0 0 0"/>
-		<parent link="${robot_id}right_hub"/>
-		<child link="${robot_id}base/joint1"/>
-	</joint>
-	<joint name="${robot_id}right_hub_joint" type="fixed">
+	<joint name="${robot_id}/base/joint1" type="fixed">
+		<origin xyz="0 0 0" rpy="0 0 0"/>
+		<parent link="${robot_id}/right_hub"/>
+		<child link="${robot_id}/base/joint1"/>
+	</joint>
+	<joint name="${robot_id}/right_hub_joint" type="fixed">
 		<origin xyz="0 -0.15 0.08" rpy="0 0 0"/>
-		<parent link="${robot_id}base_link"/>
-		<child link="${robot_id}right_hub"/>
+		<parent link="${robot_id}/base_link"/>
+		<child link="${robot_id}/right_hub"/>
 		<axis xyz="0 1 0"/>
 	</joint>
@@ -345,5 +346,5 @@
 	<bumper id="9" x="-0.1476" y="-0.1712" z="${bumper_height}" roll="0" pitch="0" yaw="${-1.5708-0.4262}" />
 <!-- ************************************************ LASER SCANER ********************************-->
-	<link name="${robot_id}laserSensors/sensor0">
+	<link name="${robot_id}/laserSensors/sensor0">
 		<inertial>
 			<mass value="0.0001"/>
@@ -362,14 +363,14 @@
     	</visual>
 	</link>
-	<gazebo reference="${robot_id}laserSensors/sensor0">
+	<gazebo reference="${robot_id}/laserSensors/sensor0">
 		<material value="Gazebo/Blue"/>
 	</gazebo>
-	<joint name="${robot_id}laserSensors/0_joint" type="fixed">
+	<joint name="${robot_id}/laserSensors/0_joint" type="fixed">
 		<origin xyz="0.1498 0 0.05" rpy="0 0 0"/>
-		<parent link="${robot_id}top_plate"/>
-		<child link="${robot_id}laserSensors/sensor0"/>
+		<parent link="${robot_id}/top_plate"/>
+		<child link="${robot_id}/laserSensors/sensor0"/>
 	</joint>
 	<!-- ************************************************ CAMERA ********************************-->
-	<link name="${robot_id}cameraSensors/sensor0">
+	<link name="${robot_id}/cameraSensors/sensor0">
 		<inertial>
 			<mass value="0.0001"/>
@@ -388,14 +389,14 @@
     	</visual>
 	</link>
-	<gazebo reference="${robot_id}cameraSensors/sensor0">
+	<gazebo reference="${robot_id}/cameraSensors/sensor0">
 		<material value="Gazebo/Blue"/>
 	</gazebo>
-	<joint name="${robot_id}cameraSensors/0_joint" type="fixed">
+	<joint name="${robot_id}/cameraSensors/0_joint" type="fixed">
 		<origin xyz="0.1498 0 0.001" rpy="1.5708 0 1.5708"/>
-		<parent link="${robot_id}top_plate"/>
-		<child link="${robot_id}cameraSensors/sensor0"/>
+		<parent link="${robot_id}/top_plate"/>
+		<child link="${robot_id}/cameraSensors/sensor0"/>
 	</joint>
 	<!-- ************************************************ GYRO ********************************-->
-	<link name="${robot_id}gyroSensors/sensor0">
+	<link name="${robot_id}/gyroSensors/sensor0">
 		<inertial>
 			<mass value="0.0001"/>
@@ -414,14 +415,14 @@
     	</visual>
 	</link>
-	<gazebo reference="${robot_id}gyroSensors/sensor0">
+	<gazebo reference="${robot_id}/gyroSensors/sensor0">
 		<material value="Gazebo/Blue"/>
 	</gazebo>
-	<joint name="${robot_id}gyroSensors/0_joint" type="fixed">
+	<joint name="${robot_id}/gyroSensors/0_joint" type="fixed">
 		<origin xyz="0 0 0.0" rpy="0 0 0"/>
-		<parent link="${robot_id}top_plate"/>
-		<child link="${robot_id}gyroSensors/sensor0"/>
+		<parent link="${robot_id}/top_plate"/>
+		<child link="${robot_id}/gyroSensors/sensor0"/>
 	</joint>
 <!-- ************************************************ ACCELEROMETER ********************************-->
-	<link name="${robot_id}accelerometerSensors/sensor0">
+	<link name="${robot_id}/accelerometerSensors/sensor0">
 		<inertial>
 			<mass value="0.0001"/>
@@ -440,11 +441,11 @@
     	</visual>
 	</link>
-	<gazebo reference="${robot_id}accelerometerSensors/sensor0">
+	<gazebo reference="${robot_id}/accelerometerSensors/sensor0">
 		<material value="Gazebo/Blue"/>
 	</gazebo>
-	<joint name="${robot_id}accelerometerSensors/0_joint" type="fixed">
+	<joint name="${robot_id}/accelerometerSensors/0_joint" type="fixed">
 		<origin xyz="0 0 0.0" rpy="0 0 0"/>
-		<parent link="${robot_id}top_plate"/>
-		<child link="${robot_id}accelerometerSensors/sensor0"/>
+		<parent link="${robot_id}/top_plate"/>
+		<child link="${robot_id}/accelerometerSensors/sensor0"/>
 	</joint>
 	<xacro:macro name="p3dx_gazebo_ext">
