Commit message: Rotation of data received from laser_scan

File: src/pioneer-p3dx/p3dx_urdf_model/defs/pioneer3dx_body.xacro (robot description, xacro)
@@ -366,5 +366,5 @@
 	</gazebo>
 	<joint name="${robot_id}laserSensors/0_joint" type="fixed">
-		<origin xyz="0.1498 0 0.05" rpy="0 0 0"/>
+		<origin xyz="0.1498 0 0.05" rpy="0 0 -1.5708"/>
 		<parent link="${robot_id}top_plate"/>
 		<child link="${robot_id}laserSensors/sensor0"/>

Commit message: Adding base_footprint odom frame support

File: src/pioneer-p3dx/p3dx_urdf_model/defs/pioneer3dx_body.xacro (robot description, xacro)
@@ -59,5 +59,10 @@
 	</xacro:macro>
 <!-- *********************************** CHASIS ********************************************** -->
-	<!-- Chassis description -->
+<!-- base_footprint -->
+	<link name="${robot_id}base_footprint"></link>
+	<gazebo reference="${robot_id}base_footprint">
+		<material value="Gazebo/Red"/>
+	</gazebo>
+<!-- Chassis description -->
 	<link name="${robot_id}base_link">
 		<!-- CHECK THESE VALUES. THEY MAY BE COMPLETELY WRONG. -->
@@ -89,4 +94,9 @@
 		<material value="Gazebo/Red"/>
 	</gazebo>
+	<joint name="base_link_joint" type="fixed">
+		<origin xyz="0 0 0" rpy="0 0 0"/>
+		<parent link="${robot_id}base_footprint"/>
+		<child link="${robot_id}base_link"/>
+	</joint>
 <!-- Top part of the robot -->
 	<link name="${robot_id}top_plate">

Commit message: FIX in coordinates of base_footprint

File: src/pioneer-p3dx/p3dx_urdf_model/defs/pioneer3dx_body.xacro (robot description, xacro)
@@ -121,5 +121,5 @@
 	</gazebo>
 	<joint name="${robot_id}base_top_joint" type="fixed">
-		<origin xyz="-0.0 0 0.24" rpy="0 0 0"/>
+		<origin xyz="0.0 0.0 0.24" rpy="0.0 0.0 0.0"/>
 		<parent link="${robot_id}base_link"/>
 		<child link="${robot_id}top_plate"/>
