Commit message: Prefifing property tags with xacro keyword

File: src/pioneer-p3dx/p3dx_urdf_model/defs/pioneer3dx.xacro (robot description, xacro)
@@ -6,5 +6,5 @@
 	   name="pioneer3dx">
 	<!--  SET ROBOT NAME -->
-    <property name="robot_id" value=""/>
+    <xacro:property name="robot_id" value=""/>
     <xacro:include filename="$(find p3dx_urdf_model)/defs/pioneer3dx_body.xacro" />
 	<!-- <xacro:right_wheel_joint suffix="" reflect="1"/>

File: src/pioneer-p3dx/p3dx_urdf_model/defs/pioneer3dx_body.xacro (robot description, xacro)
@@ -322,5 +322,5 @@
 <!-- ******************************SONARS**************************************************** -->
 	<!-- front side sonars -->
-	<property name="sonar_height" value="+0.21"/>
+	<xacro:property name="sonar_height" value="+0.21"/>
 	<sonar id="0" x="0.1064" y="-0.1381" z="${sonar_height}" roll="0" pitch="0" yaw="-1.5708" />
 	<sonar id="1" x="0.1555" y="-0.1202" z="${sonar_height}" roll="0" pitch="0" yaw="${-1.5708+0.6981}" />
@@ -342,5 +342,5 @@
 	<!-- *************************BUMPERS****************************************************** -->
 	<!-- front side bumpers -->
-	<property name="bumper_height" value="+0.0681"/>
+	<xacro:property name="bumper_height" value="+0.0681"/>
 	<bumper id="0" x="+0.1767" y="-0.1700" z="${bumper_height}" roll="0" pitch="0" yaw="${-1.5708+0.6210}" />
 	<bumper id="1" x="+0.2377" y="-0.0909" z="${bumper_height}" roll="0" pitch="0" yaw="${-1.5708+1.2318}" />
@@ -349,5 +349,5 @@
 	<bumper id="4" x="+0.1767" y="+0.1700" z="${bumper_height}" roll="0" pitch="0" yaw="${1.5708-0.6007}" />
 	<!-- back side bumpers -->
-	<property name="bumper_height" value="+0.0681"/>
+	<xacro:property name="bumper_height" value="+0.0681"/>
 	<bumper id="5" x="-0.1476" y="+0.1712" z="${bumper_height}" roll="0" pitch="0" yaw="${1.5708+0.4465}" />
 	<bumper id="6" x="-0.2259" y="+0.0978" z="${bumper_height}" roll="0" pitch="0" yaw="${1.5708+1.0573}" />
